File: badge2.sch (EAGLE design)
At the start: 78 parts, among them IC1 ESP32-PICO-D4, Q1 CJ2302, Q2 CJ2302, Q3 FDN340P, Q4 CJ2302, U2 STM32F103CBT6, U3 MCP73831, Y1 8MHz

Commit message: Added license
Parts:
- added LOGO1: OSHW-LOGOM, SparkFun-Aesthetics:OSHW-LOGOM
- C14: device Seeed-Capacitor:CERAMIC-10UF-10V-10%-X5R(0603) -> Seeed-Capacitor:CERAMIC-4.7UF-10V-10%-X5R(0603)
- R3: value 2K -> 1.5K
- R8: device Seeed-Resistor:SMD-RES-10K-5%-1/10W(0603) -> Seeed-Resistor:SMD-RES-10K-1%-1/10W(0603)
Other:
- note added: "1337 3310 WiFi motherboard Mastro Gippo 2018"
